File: WETHAP_PCB/WETHAP_PCB.kicad_sch (KiCad schematic)
At the start: 7 parts, among them J1 Conn_01x20_Socket, J2 Conn_01x20_Socket

Commit message: pcb v0.2.0
Parts:
- added LPS25HB1, LPS25HB2: Conn_01x04_Socket, Connector_PinSocket_2.54mm:PinSocket_1x04_P2.54mm_Vertical, symbol Connector:Conn_01x04_Socket
Connections:
- net gnd: now also LPS25HB1.4 (Pin_4), LPS25HB2.8 (Pin_4)
- net scl: now also LPS25HB1.2 (Pin_2)
- net sda: now also LPS25HB1.3 (Pin_3)
- net vbus: now also LPS25HB1.1 (Pin_1), LPS25HB2.5 (Pin_1)
Changed lines of the file:
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@@
+    (stroke (width 0) (type default))
+  )
+  (wire (pts (xy 177.8 130.81) (xy 195.58 130.81))
     (stroke (width 0) (type default))
   )
@@
     (stroke (width 0) (type default))
   )
+  (wire (pts (xy 185.42 133.35) (xy 195.58 133.35))
+    (stroke (width 0) (type default))
+  )
   (wire (pts (xy 195.58 101.6) (xy 203.2 101.6))
     (stroke (width 0) (type default))
@@
     (stroke (width 0) (type default))
   )
+  (wire (pts (xy 195.58 135.89) (xy 190.5 135.89))
+    (stroke (width 0) (type default))
+  )
   (wire (pts (xy 124.46 102.87) (xy 130.81 102.87))
     (stroke (width 0) (type default))
@@
     (stroke (width 0) (type default))
   )
+  (wire (pts (xy 205.74 135.89) (xy 219.71 135.89))
+    (stroke (width 0) (type default))
+  )
+  (wire (pts (xy 185.42 128.27) (xy 195.58 128.27))
+    (stroke (width 0) (type default))
+  )
+  (wire (pts (xy 205.74 128.27) (xy 213.36 128.27))
+    (stroke (width 0) (type default))
+  )
   (wire (pts (xy 101.6 77.47) (xy 105.41 77.47))
     (stroke (width 0) (type default))
@@
     )
   )
+  (global_label "sda" (shape input) (at 185.42 133.35 180) (fields_autoplaced)
+    (effects (font (size 1.27 1.27)) (justify right))
+    (property "Intersheetrefs" "${INTERSHEET_REFS}" (at 179.1087 133.35 0)
+      (effects (font (size 1.27 1.27)) (justify right) hide)
+    )
+  )
   (global_label "sda" (shape input) (at 130.81 120.65 0) (fields_autoplaced)
     (effects (font (size 1.27 1.27)) (justify left))
@@
     )
   )
+  (global_label "vbus" (shape input) (at 219.71 135.89 0) (fields_autoplaced)
+    (effects (font (size 1.27 1.27)) (justify left))
+    (property "Intersheetrefs" "${INTERSHEET_REFS}" (at 226.9889 135.89 0)
+      (effects (font (size 1.27 1.27)) (justify left) hide)
+    )
+  )
   (global_label "gnd" (shape input) (at 101.6 90.17 180) (fields_autoplaced)
     (effects (font (size 1.27 1.27)) (justify right))
@@
     )
   )
+  (global_label "scl" (shape input) (at 177.8 130.81 180) (fields_autoplaced)
+    (effects (font (size 1.27 1.27)) (justify right))
+    (property "Intersheetrefs" "${INTERSHEET_REFS}" (at 172.0329 130.81 0)
+      (effects (font (size 1.27 1.27)) (justify right) hide)
+    )
+  )
   (global_label "gnd" (shape input) (at 201.93 76.2 180) (fields_autoplaced)
     (effects (font (size 1.27 1.27)) (justify right))
@@
     )
   )
+  (global_label "vbus" (shape input) (at 185.42 128.27 180) (fields_autoplaced)
+    (effects (font (size 1.27 1.27)) (justify right))
+    (property "Intersheetrefs" "${INTERSHEET_REFS}" (at 178.1411 128.27 0)
+      (effects (font (size 1.27 1.27)) (justify right) hide)
+    )
+  )
   (global_label "vbus" (shape input) (at 195.58 78.74 180) (fields_autoplaced)
     (effects (font (size 1.27 1.27)) (justify right))
@@
     )
   )
+  (global_label "gnd" (shape input) (at 213.36 128.27 0) (fields_autoplaced)
+    (effects (font (size 1.27 1.27)) (justify left))
+    (property "Intersheetrefs" "${INTERSHEET_REFS}" (at 219.7922 128.27 0)
+      (effects (font (size 1.27 1.27)) (justify left) hide)
+    )
+  )
   (global_label "scl" (shape input) (at 201.93 81.28 180) (fields_autoplaced)
     (effects (font (size 1.27 1.27)) (justify right))
@@
     (effects (font (size 1.27 1.27)) (justify right))
     (property "Intersheetrefs" "${INTERSHEET_REFS}" (at 188.3011 101.6 0)
+      (effects (font (size 1.27 1.27)) (justify right) hide)
+    )
+  )
+  (global_label "gnd" (shape input) (at 190.5 135.89 180) (fields_autoplaced)
+    (effects (font (size 1.27 1.27)) (justify right))
+    (property "Intersheetrefs" "${INTERSHEET_REFS}" (at 184.0678 135.89 0)
       (effects (font (size 1.27 1.27)) (justify right) hide)
     )
@@
     )
   )
+  (symbol (lib_id "Connector:Conn_01x04_Socket") (at 190.5 130.81 0) (mirror y) (unit 1)
+    (in_bom yes) (on_board yes) (dnp no)
+    (property "Reference" "LPS25HB1" (at 189.23 130.81 0)
+      (effects (font (size 1.27 1.27)) (justify left))
+    )
+    (property "Value" "Conn_01x04_Socket" (at 189.23 133.35 0)
+      (effects (font (size 1.27 1.27)) (justify left))
+    )
+    (property "Footprint" "Connector_PinSocket_2.54mm:PinSocket_1x04_P2.54mm_Vertical" (at 190.5 130.81 0)
+      (effects (font (size 1.27 1.27)) hide)
+    )
+    (property "Datasheet" "~" (at 190.5 130.81 0)
+      (effects (font (size 1.27 1.27)) hide)
+    )
+    (pin "1")
+    (pin "2")
+    (pin "3")
+    (pin "4")
+    (instances
+      (project "WETHAP_PCB"
+        (path "/1fd4f93a-1ad9-4679-87e3-0672e9ca2f50"
+          (reference "LPS25HB1") (unit 1)
+        )
+      )
+    )
+  )
   (symbol (lib_id "Connector:Conn_01x04_Socket") (at 208.28 78.74 0) (unit 1)
     (in_bom yes) (on_board yes) (dnp no) (fields_autoplaced)
@@
         )
       )
+    )
+  )
+  (symbol (lib_name "Conn_01x04_Socket_1") (lib_id "Connector:Conn_01x04_Socket") (at 210.82 133.35 0) (mirror x) (unit 1)
+    (in_bom yes) (on_board yes) (dnp no)
+    (property "Reference" "LPS25HB2" (at 212.09 133.35 0)
+      (effects (font (size 1.27 1.27)) (justify left))
+    )
+    (property "Value" "Conn_01x04_Socket" (at 212.09 130.81 0)
+      (effects (font (size 1.27 1.27)) (justify left))
+    )
+    (property "Footprint" "Connector_PinSocket_2.54mm:PinSocket_1x04_P2.54mm_Vertical" (at 210.82 133.35 0)
+      (effects (font (size 1.27 1.27)) hide)
+    )
+    (property "Datasheet" "~" (at 210.82 133.35 0)
+      (effects (font (size 1.27 1.27)) hide)
+    )
+    (pin "5")
+    (pin "6")
+    (pin "7")
+    (pin "8")
+    (instances
+      (project "WETHAP_PCB"
+        (path "/1fd4f93a-1ad9-4679-87e3-0672e9ca2f50"
+          (reference "LPS25HB2") (unit 1)
+        )
+      )

Commit message: fix circuit
Connections:
- net scl: now also DHT20.4 (Pin_4); no longer DHT20.2 (Pin_2)
- net sda: now also DHT20.2 (Pin_2); no longer DHT20.4 (Pin_4)
Changed lines of the file:
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@@
+    )
+  )
+  (global_label "scl" (shape input) (at 201.93 105.41 180) (fields_autoplaced)
+    (effects (font (size 1.27 1.27)) (justify right))
+    (property "Intersheetrefs" "${INTERSHEET_REFS}" (at 196.1629 105.41 0)
+      (effects (font (size 1.27 1.27)) (justify right) hide)
     )
   )
@@
     )
   )
-  (global_label "sda" (shape input) (at 201.93 105.41 180) (fields_autoplaced)
+  (global_label "sda" (shape input) (at 201.93 110.49 180) (fields_autoplaced)
     (effects (font (size 1.27 1.27)) (justify right))
-    (property "Intersheetrefs" "${INTERSHEET_REFS}" (at 195.6187 105.41 0)
+    (property "Intersheetrefs" "${INTERSHEET_REFS}" (at 195.6187 110.49 0)
       (effects (font (size 1.27 1.27)) (justify right) hide)
     )
@@
       (effects (font (size 1.27 1.27)) (justify right) hide)
     )
-  )
-  (global_label "scl" (shape input) (at 201.93 110.49 180) (fields_autoplaced)
-    (effects (font (size 1.27 1.27)) (justify right))
-    (property "Intersheetrefs" "${INTERSHEET_REFS}" (at 196.1629 110.49 0)
-      (effects (font (size 1.27 1.27)) (justify right) hide)
-    )

Commit message: websocket
Parts:
- removed BME680: Conn_01x04_Socket, Connector_PinHeader_2.54mm:PinHeader_1x04_P2.54mm_Vertical, symbol Connector:Conn_01x04_Socket
- added H1, H2, H3, H4: MountingHole_Pad, MountingHole:MountingHole_3.2mm_M3_DIN965_Pad, symbol Mechanical:MountingHole_Pad
Connections:
- net adc_vref: now also J2.15 (Pin_15), RV1.3, RV2.3; no longer J2.6 (Pin_6), RV1.1, RV2.1
- net gnd: now also RV1.1, RV2.1, H1.1, H2.1, H3.1, H4.1; no longer RV1.3, RV2.3
- net scl: now also J2.2 (Pin_2); no longer J2.19 (Pin_19)
- net sda: now also J2.1 (Pin_1); no longer J2.20 (Pin_20)
- net vbus: now also J2.20 (Pin_20); no longer J2.1 (Pin_1)
- net at J2.10 (Pin_10): no longer RV1.2
- net ADC0: now reaches J2.11 (Pin_11)
- net ADC0: now also RV1.2
- net ADC1: now reaches J2.12 (Pin_12)
- net ADC1: now also RV2.2
- net at J2.9 (Pin_9): no longer RV2.2
- no-connect marks 0 -> 28
Other:
- note added: "Adjust info"
- note added: "Display"
- note added: "Hole"
- note added: "Raspberry Pi Pico W"
- note added: "Sensors"
- moved on the sheet: DHT20, J1, J2, LPS25HB1, LPS25HB2, RV1, RV2, SSD1306
